File: PCB design/Chessbot_v7.sch (EAGLE design)
At the start: 28 parts, among them Q1 PMV16XNR

Commit message: Minor design alterations
Parts:
- added B1: (no value), ME507:BEAD0805
Connections:
- net 3V3: now also B1.1, B1.2
Changed lines of the file:
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@@
 <part name="TCRT5000" library="Connector" library_urn="urn:adsk.eagle:library:16378166" deviceset="PINHD-2X2" device="" package3d_urn="urn:adsk.eagle:package:22455/2"/>
 <part name="ELECTROMAGNET" library="Connector" library_urn="urn:adsk.eagle:library:16378166" deviceset="PINHD-1X2" device="" package3d_urn="urn:adsk.eagle:package:22435/2"/>
+<part name="B1" library="ME507" deviceset="BEAD" device="0805"/>
 </parts>
 <sheets>
@@
 <attribute name="VALUE" x="25.4" y="177.165" size="1.778" layer="96" rot="R180" align="center"/>
 </instance>
-<instance part="SUPPLY15" gate="G$1" x="86.36" y="149.86" smashed="yes" rot="MR0">
-<attribute name="VALUE" x="86.36" y="154.305" size="1.778" layer="96" rot="MR180" align="center"/>
+<instance part="SUPPLY15" gate="G$1" x="86.36" y="162.56" smashed="yes" rot="MR0">
+<attribute name="VALUE" x="86.36" y="167.005" size="1.778" layer="96" rot="MR180" align="center"/>
 </instance>
 <instance part="SUPPLY16" gate="G$1" x="76.2" y="104.14" smashed="yes">
@@
 <attribute name="NAME" x="222.25" y="169.799" size="1.778" layer="95"/>
 <attribute name="VALUE" x="222.25" y="156.464" size="1.778" layer="96"/>
+</instance>
+<instance part="B1" gate="G$1" x="86.36" y="154.94" smashed="yes" rot="R90">
+<attribute name="NAME" x="82.55" y="151.13" size="1.778" layer="95" rot="R90"/>
+<attribute name="VALUE" x="92.71" y="151.13" size="1.778" layer="96" rot="R90"/>
 </instance>
 </instances>
@@
 </segment>
 <segment>
-<pinref part="SUPPLY15" gate="G$1" pin="VCC"/>
-<pinref part="LED1" gate="G$1" pin="A"/>
-<wire x1="86.36" y1="134.62" x2="86.36" y2="149.86" width="0.1524" layer="91"/>
-<wire x1="86.36" y1="149.86" x2="99.06" y2="149.86" width="0.1524" layer="91"/>
-<wire x1="99.06" y1="149.86" x2="99.06" y2="144.78" width="0.1524" layer="91"/>
-<junction x="86.36" y="149.86"/>
-<pinref part="C3" gate="G$1" pin="1"/>
-<wire x1="66.04" y1="147.32" x2="66.04" y2="149.86" width="0.1524" layer="91"/>
-<wire x1="66.04" y1="149.86" x2="86.36" y2="149.86" width="0.1524" layer="91"/>
-<pinref part="U$2" gate="G$1" pin="VCC"/>
-<wire x1="76.2" y1="129.54" x2="76.2" y2="134.62" width="0.1524" layer="91"/>
-<pinref part="R8" gate="G$1" pin="2"/>
-<wire x1="76.2" y1="134.62" x2="86.36" y2="134.62" width="0.1524" layer="91"/>
-<wire x1="86.36" y1="134.62" x2="88.9" y2="134.62" width="0.1524" layer="91"/>
-<wire x1="88.9" y1="134.62" x2="88.9" y2="132.08" width="0.1524" layer="91"/>
-<junction x="86.36" y="134.62"/>
-</segment>
-<segment>
 <pinref part="R6" gate="G$1" pin="2"/>
 <pinref part="SUPPLY25" gate="G$1" pin="VCC"/>
@@
 <wire x1="176.53" y1="90.932" x2="176.53" y2="88.392" width="0.1524" layer="91"/>
 </segment>
-</net>
+<segment>
+<pinref part="LED1" gate="G$1" pin="A"/>
+<wire x1="86.36" y1="134.62" x2="86.36" y2="149.86" width="0.1524" layer="91"/>
+<wire x1="86.36" y1="149.86" x2="86.36" y2="160.02" width="0.1524" layer="91"/>
+<wire x1="99.06" y1="149.86" x2="99.06" y2="144.78" width="0.1524" layer="91"/>
+<pinref part="C3" gate="G$1" pin="1"/>
+<wire x1="66.04" y1="147.32" x2="66.04" y2="149.86" width="0.1524" layer="91"/>
+<pinref part="U$2" gate="G$1" pin="VCC"/>
+<wire x1="76.2" y1="129.54" x2="76.2" y2="134.62" width="0.1524" layer="91"/>
+<pinref part="R8" gate="G$1" pin="2"/>
+<wire x1="76.2" y1="134.62" x2="86.36" y2="134.62" width="0.1524" layer="91"/>
+<wire x1="86.36" y1="134.62" x2="88.9" y2="134.62" width="0.1524" layer="91"/>
+<wire x1="88.9" y1="134.62" x2="88.9" y2="132.08" width="0.1524" layer="91"/>
+<junction x="86.36" y="134.62"/>
+<wire x1="66.04" y1="149.86" x2="86.36" y2="149.86" width="0.1524" layer="91"/>
+<junction x="86.36" y="149.86"/>
+<wire x1="86.36" y1="149.86" x2="99.06" y2="149.86" width="0.1524" layer="91"/>
+<pinref part="B1" gate="G$1" pin="1"/>
+<junction x="86.36" y="149.86"/>
+<pinref part="B1" gate="G$1" pin="2"/>
+<pinref part="SUPPLY15" gate="G$1" pin="VCC"/>
+<wire x1="86.36" y1="162.56" x2="86.36" y2="160.02" width="0.1524" layer="91"/>
+<junction x="86.36" y="160.02"/>
+</segment>
+</net>
