File: PCB design/Chessbot_v7.brd (EAGLE design)
At the start: 59.7 x 82.2 mm, 28 parts, among them Q1 PMV16XNR

Commit message: Minor design alterations
Parts:
- added B1: (no value), ME507:0805
Connections:
- net 3V3: now also B1.1, B1.2
Routing:
- net 3V3: track 155.4 -> 144.9 mm
Changed lines of the file:
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@@
 <wire x1="59.67" y1="82.22" x2="0" y2="82.22" width="0" layer="20"/>
 <wire x1="0" y1="82.22" x2="0" y2="0" width="0" layer="20"/>
-<text x="39.624" y="74.549" size="1.27" layer="25">Chessbot v7
+<text x="39.751" y="74.041" size="1.27" layer="25">Chessbot v7
 Hudson, Dunn, Ruiz</text>
 <text x="33.909" y="78.994" size="0.8128" layer="25">GND
@@
 </element>
 <element name="C2" library="rcl" library_urn="urn:adsk.eagle:library:334" package="E2,5-6" package3d_urn="urn:adsk.eagle:package:23349/1" value="100uF" x="4.572" y="21.59" smashed="yes" rot="R270">
-<attribute name="NAME" x="7.366" y="20.193" size="0.8128" layer="25" ratio="10" rot="R270"/>
+<attribute name="NAME" x="7.366" y="20.193" size="0.8128" layer="25" ratio="10"/>
 <attribute name="POPULARITY" value="14" x="-110.998" y="-11.43" size="1.778" layer="27" rot="R270" display="off"/>
 <attribute name="SPICEPREFIX" value="C" x="-110.998" y="-11.43" size="1.778" layer="27" rot="R270" display="off"/>
-<attribute name="VALUE" x="9.017" y="20.447" size="0.8128" layer="27" ratio="10" rot="R270"/>
+<attribute name="VALUE" x="7.239" y="19.05" size="0.8128" layer="27" ratio="10"/>
 </element>
 <element name="C3" library="rcl" library_urn="urn:adsk.eagle:library:334" package="C0805" package3d_urn="urn:adsk.eagle:package:23617/2" value="0.1uF" x="22.352" y="73.914" smashed="yes" rot="R180">
@@
 <attribute name="THERMALLOSS" value="" x="51.943" y="7.62" size="1.778" layer="27" rot="R90" display="off"/>
 <attribute name="TYPE" value="" x="51.943" y="7.62" size="1.778" layer="27" rot="R90" display="off"/>
+</element>
+<element name="B1" library="ME507" package="0805" value="" x="49.53" y="52.07" smashed="yes">
+<attribute name="NAME" x="48.53" y="52.945" size="1.016" layer="25"/>
+<attribute name="VALUE" x="48.53" y="50.17" size="1.016" layer="27"/>
 </element>
 </elements>
@@
 <contactref element="ESP32" pad="P1"/>
 <contactref element="R2" pad="2"/>
-<contactref element="LED1" pad="A"/>
 <contactref element="R6" pad="2"/>
 <contactref element="R7" pad="2"/>
@@
 <contactref element="C4" pad="1"/>
 <contactref element="DRIVER2" pad="JP2_7"/>
-<contactref element="C3" pad="1"/>
-<contactref element="U$2" pad="8"/>
-<contactref element="R8" pad="2"/>
 <contactref element="C5" pad="1"/>
 <wire x1="8.001" y1="38.166" x2="10.16" y2="38.166" width="1.016" layer="1"/>
@@
 <wire x1="15.24" y1="52.07" x2="15.24" y2="62.23" width="0.8128" layer="1"/>
 <wire x1="12.7" y1="64.77" x2="15.24" y2="62.23" width="0.8128" layer="1"/>
-<wire x1="54.61" y1="68.58" x2="54.61" y2="69.85" width="0.8128" layer="1"/>
-<wire x1="54.61" y1="69.85" x2="53.34" y2="71.12" width="0.8128" layer="1"/>
-<wire x1="23.302" y1="70.292" x2="23.302" y2="71.12" width="0.8128" layer="1"/>
-<wire x1="23.302" y1="71.12" x2="23.302" y2="73.914" width="0.8128" layer="1"/>
-<wire x1="23.302" y1="73.914" x2="23.302" y2="77.47" width="0.8128" layer="1"/>
 <wire x1="54.61" y1="68.58" x2="57.15" y2="66.04" width="0.3048" layer="1"/>
 <wire x1="57.15" y1="66.04" x2="57.15" y2="62.23" width="0.3048" layer="1"/>
@@
 <wire x1="57.15" y1="55.88" x2="55.88" y2="54.61" width="0.3048" layer="1"/>
 <wire x1="53.34" y1="54.61" x2="55.88" y2="54.61" width="0.3048" layer="1"/>
-<wire x1="52.385" y1="60.64" x2="41.021" y2="60.64" width="0.3048" layer="1"/>
 <wire x1="57.15" y1="62.23" x2="53.975" y2="62.23" width="0.3048" layer="1"/>
 <wire x1="53.975" y1="62.23" x2="52.385" y2="60.64" width="0.3048" layer="1"/>
-<wire x1="7.899" y1="66.04" x2="11.43" y2="66.04" width="0.3048" layer="1"/>
-<wire x1="12.7" y1="64.77" x2="11.43" y2="66.04" width="0.8128" layer="1"/>
+<wire x1="12.7" y1="64.77" x2="11.197" y2="66.273" width="0.8128" layer="1"/>
 <wire x1="5.08" y1="69.85" x2="7.899" y2="67.031" width="0.3048" layer="1"/>
-<wire x1="7.899" y1="67.031" x2="7.899" y2="66.04" width="0.3048" layer="1"/>
 <wire x1="26.609" y1="76.708" x2="26.609" y2="74.168" width="0.3048" layer="1"/>
-<wire x1="45.023" y1="49.355" x2="45.023" y2="48.957" width="0.3048" layer="1"/>
-<wire x1="45.023" y1="48.957" x2="45.72" y2="48.26" width="0.3048" layer="1"/>
-<wire x1="45.72" y1="48.26" x2="46.99" y2="48.26" width="0.3048" layer="1"/>
-<wire x1="46.99" y1="48.26" x2="53.34" y2="54.61" width="0.3048" layer="1"/>
 <wire x1="15.24" y1="62.23" x2="17.78" y2="64.77" width="0.8128" layer="1"/>
 <wire x1="17.78" y1="64.77" x2="17.78" y2="67.31" width="0.8128" layer="1"/>
 <wire x1="17.78" y1="67.31" x2="19.05" y2="68.58" width="0.8128" layer="1"/>
 <wire x1="19.05" y1="68.58" x2="21.59" y2="68.58" width="0.8128" layer="1"/>
-<wire x1="21.59" y1="68.58" x2="23.302" y2="70.292" width="0.8128" layer="1"/>
-<wire x1="53.34" y1="71.12" x2="23.302" y2="71.12" width="0.8128" layer="1"/>
-<wire x1="11.43" y1="66.04" x2="11.197" y2="66.273" width="0.8128" layer="1"/>
 <wire x1="10.48" y1="68.45654375" x2="10.48" y2="70.612" width="0.8128" layer="1"/>
 <wire x1="11.197" y1="66.273" x2="11.197" y2="67.73954375" width="0.8128" layer="1"/>
 <wire x1="11.197" y1="67.73954375" x2="10.48" y2="68.45654375" width="0.8128" layer="1"/>
-<wire x1="23.302" y1="73.914" x2="26.355" y2="73.914" width="0.8128" layer="1"/>
 <wire x1="26.355" y1="73.914" x2="26.609" y2="74.168" width="0.8128" layer="1"/>
+<contactref element="LED1" pad="A"/>
+<contactref element="C3" pad="1"/>
+<contactref element="U$2" pad="8"/>
+<contactref element="R8" pad="2"/>
+<contactref element="B1" pad="1"/>
+<contactref element="B1" pad="2"/>
+<wire x1="45.023" y1="49.355" x2="45.61" y2="48.768" width="0.3048" layer="1"/>
+<wire x1="45.61" y1="48.768" x2="46.228" y2="48.768" width="0.3048" layer="1"/>
+<wire x1="46.228" y1="48.768" x2="48.53" y2="51.07" width="0.3048" layer="1"/>
+<wire x1="48.53" y1="51.07" x2="48.53" y2="52.07" width="0.3048" layer="1"/>
+<wire x1="50.53" y1="52.07" x2="50.8" y2="52.07" width="0.3048" layer="1"/>
+<wire x1="50.8" y1="52.07" x2="53.34" y2="54.61" width="0.3048" layer="1"/>
+<wire x1="21.59" y1="68.58" x2="24.13" y2="71.12" width="0.8128" layer="1"/>
+<wire x1="24.13" y1="71.12" x2="33.02" y2="71.12" width="0.8128" layer="1"/>
+<wire x1="33.02" y1="71.12" x2="34.29" y2="72.39" width="0.8128" layer="1"/>
+<wire x1="34.29" y1="72.39" x2="38.1" y2="72.39" width="0.8128" layer="1"/>
+<wire x1="38.1" y1="72.39" x2="38.1" y2="77.47" width="0.8128" layer="1"/>
+<wire x1="38.1" y1="77.47" x2="39.37" y2="78.74" width="0.8128" layer="1"/>
+<wire x1="39.37" y1="78.74" x2="55.88" y2="78.74" width="0.8128" layer="1"/>
+<wire x1="55.88" y1="78.74" x2="57.15" y2="77.47" width="0.8128" layer="1"/>
+<wire x1="57.15" y1="77.47" x2="57.15" y2="71.12" width="0.8128" layer="1"/>
+<wire x1="57.15" y1="71.12" x2="54.61" y2="68.58" width="0.8128" layer="1"/>
+<wire x1="26.609" y1="76.708" x2="23.302" y2="77.47" width="0" layer="19" extent="1-1"/>
+<wire x1="23.302" y1="73.914" x2="26.355" y2="73.914" width="0" layer="19" extent="1-1"/>
+<wire x1="10.48" y1="70.612" x2="23.302" y2="73.914" width="0" layer="19" extent="1-1"/>
+<wire x1="48.53" y1="52.07" x2="50.53" y2="52.07" width="0" layer="19" extent="1-1"/>
+<wire x1="7.899" y1="67.031" x2="10.48" y2="70.612" width="0" layer="19" extent="1-1"/>
+<wire x1="7.899" y1="66.04" x2="7.899" y2="67.031" width="0" layer="19" extent="1-1"/>
+<wire x1="41.021" y1="60.64" x2="52.385" y2="60.64" width="0" layer="19" extent="1-1"/>
 </signal>
 <signal name="N$14">

Commit message: DRC passed, CAM files
Routing:
- net 3V3: track 144.9 -> 172.4 mm
- net N$14: track 37.4 -> 38.3 mm
